File: LogicAnalyzer/LogicAnalyzer.kicad_pcb (KiCad board)
At the start: 2 copper layers, 55 x 65 mm, 29 parts, among them J1 Conn_02x03_Odd_Even, J2 Connector, J3 Chain, U1 TXB0104PW, U2 TXB0104PW, U3 TXB0104PW, U4 TXB0104PW, U5 TXB0104PW, U6 TXB0104PW, U7 Pico

Commit message: PCB update
Parts:
- added G***: LOGO, Eigene:logo, F.Cu at (198.4, 123.2)
- added REF**: WEEE-Logo_4.2x6mm_SilkScreen, Symbol:WEEE-Logo_4.2x6mm_SilkScreen, F.Cu at (180.8, 125.0)
- added REF**: OSHW-Logo2_9.8x8mm_SilkScreen, Symbol:OSHW-Logo2_9.8x8mm_SilkScreen, F.Cu at (187.9, 123.4)
- added REF**: ESD-Logo_6.6x6mm_SilkScreen, Symbol:ESD-Logo_6.6x6mm_SilkScreen, F.Cu at (180.8, 118.4)
Other:
- board text added: "Adaptation by Synthron: https://github.com/Synthron/LogicAnalyzer"
- board text added: "By El Dr. Gusman - 2024"
- board text added: "LogicAnalyzer"
- board text added: "https://github.com/gusmanb/logicanalyzer"
