File: LogicAnalyzer/LogicAnalyzer.kicad_pcb (KiCad board)
At the start: 2 copper layers, 55 x 65 mm, 33 parts, among them J1 Conn_02x03_Odd_Even, J2 Connector, J3 Chain, U1 TXB0104PW, U2 TXB0104PW, U3 TXB0104PW, U4 TXB0104PW, U5 TXB0104PW, U6 TXB0104PW, U7 Pico

Commit message: DRC Check
Parts:
- removed H4: MountingHole, MountingHole:MountingHole_3.2mm_M3_DIN965
Routing:
- net GND: vias 246 -> 283

Commit message: Brutzler Review
Parts:
- added G***: LOGO, TheBrutzlers_Lib:approved_theBrutzler, F.Cu at (193.5, 102.5)
- U1, U2, U3, U4, U5, U6: value TXB0104PW -> TXU0104PW
Routing:
- net /OUT_2: track 23.8 -> 36.0 mm
- net /OUT_1: track 24.7 -> 35.7 mm
- net /OUT_6: track 24.0 -> 33.3 mm, vias 0 -> 1
- net /OUT_4: track 24.0 -> 33.3 mm, vias 0 -> 1
- net /OUT_3: track 24.0 -> 33.2 mm, vias 0 -> 1
- net /OUT_7: track 24.4 -> 33.1 mm, vias 0 -> 1
- net /OUT_11: track 24.3 -> 33.0 mm, vias 0 -> 1
- net /OUT_12: track 24.6 -> 33.2 mm, vias 0 -> 1
- net /OUT_10: track 25.0 -> 33.4 mm, vias 0 -> 1
- net /OUT_9: track 24.9 -> 33.2 mm, vias 0 -> 1
- net /OUT_8: track 24.9 -> 33.1 mm, vias 0 -> 1
- net /OUT_5: track 25.0 -> 33.3 mm, vias 0 -> 1
- net /IN_11: track 8.12 -> 15.1 mm, vias 0 -> 1
- net /IN_10: track 8.27 -> 15.1 mm, vias 0 -> 1
- net /IN_22: track 11.1 -> 17.6 mm, vias 1 -> 0
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Other:
- copper layers 2 -> 4

Commit message: add gerbers
Routing:
- added copper zone on In1.Cu, net GND
- added copper zone on In2.Cu, net GND
Changed lines of the file:
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@@
 			(plot_on_all_layers_selection 0x0000000_00000000)
 			(disableapertmacros no)
-			(usegerberextensions no)
-			(usegerberattributes yes)
-			(usegerberadvancedattributes yes)
-			(creategerberjobfile yes)
+			(usegerberextensions yes)
+			(usegerberattributes no)
+			(usegerberadvancedattributes no)
+			(creategerberjobfile no)
 			(dashed_line_dash_ratio 12.000000)
 			(dashed_line_gap_ratio 3.000000)
@@
 			(psa4output no)
 			(plotreference yes)
-			(plotvalue yes)
+			(plotvalue no)
 			(plotfptext yes)
 			(plotinvisibletext no)
 			(sketchpadsonfab no)
-			(subtractmaskfromsilk no)
+			(subtractmaskfromsilk yes)
 			(outputformat 1)
 			(mirror no)
-			(drillshape 1)
+			(drillshape 0)
 			(scaleselection 1)
-			(outputdirectory "")
+			(outputdirectory "LA_Gerber/")
 		)
 	)
@@
 			)
 		)
-		(fp_text user "ADC_VREF"
+		(fp_text user "ADC_VRF"
 			(at 14 -12.5 45)
 			(layer "F.SilkS")
@@
 		(net 1)
 		(net_name "GND")
-		(layers "F&B.Cu")
+		(layers "F.Cu" "In1.Cu" "In2.Cu" "B.Cu")
 		(hatch edge 0.5)
 		(connect_pads
